Commit message: testing and small changes in urdf and service

File: src/arm_service/arm_service/armpi_fpv.urdf (robot description, URDF)
Before this commit: robot armpi_fpv, 15 links, 14 joints
Joints:
- joint joint1: limit lower=0.1 upper=4.15 effort=1000 velocity=10 -> lower=-0.5 upper=0.5 effort=1000 velocity=10
- joint joint2: limit lower=-1.57 upper=1.57 effort=1000 velocity=10 -> lower=-1.0 upper=1.0 effort=1000 velocity=10
- joint joint3: limit lower=-2.09 upper=2.09 effort=1000 velocity=10 -> lower=-1.06 upper=1.06 effort=1000 velocity=10

Commit message: changes to arm

File: src/arm_service/arm_service/armpi_fpv.urdf (robot description, URDF)
Before this commit: robot armpi_fpv, 15 links, 14 joints
Links:
- link base_link: geometry collision mesh filename=package://arm_service/meshes/base_link.STL; visual mesh filename=package://arm_service/meshes/base_link.STL
- link camera_link: geometry collision mesh filename=package://arm_service/meshes/camera_link.STL; visual mesh filename=package://arm_service/meshes/camera_link.STL
- link gripper_base: geometry collision mesh filename=package://arm_service/meshes/gripper_base.STL; visual mesh filename=package://arm_service/meshes/gripper_base.STL
- link l_in_link: geometry collision mesh filename=package://arm_service/meshes/l_in_link.STL; visual mesh filename=package://arm_service/meshes/l_in_link.STL
- link l_link: geometry collision mesh filename=package://arm_service/meshes/l_link.STL; visual mesh filename=package://arm_service/meshes/l_link.STL
- link l_out_link: geometry collision mesh filename=package://arm_service/meshes/l_out_link.STL; visual mesh filename=package://arm_service/meshes/l_out_link.STL
- link link1: geometry collision mesh filename=package://arm_service/meshes/link1.STL; visual mesh filename=package://arm_service/meshes/link1.STL
- link link2: geometry collision mesh filename=package://arm_service/meshes/link2.STL; visual mesh filename=package://arm_service/meshes/link2.STL
- link link3: geometry collision mesh filename=package://arm_service/meshes/link3.STL; visual mesh filename=package://arm_service/meshes/link3.STL
- link link4: geometry collision mesh filename=package://arm_service/meshes/link4.STL; visual mesh filename=package://arm_service/meshes/link4.STL
- link link5: geometry collision mesh filename=package://arm_service/meshes/link5.STL; visual mesh filename=package://arm_service/meshes/link5.STL
- link r_in_link: geometry collision mesh filename=package://arm_service/meshes/r_in_link.STL; visual mesh filename=package://arm_service/meshes/r_in_link.STL
- link r_link: geometry collision mesh filename=package://arm_service/meshes/r_link.STL; visual mesh filename=package://arm_service/meshes/r_link.STL
- link r_out_link: geometry collision mesh filename=package://arm_service/meshes/r_out_link.STL; visual mesh filename=package://arm_service/meshes/r_out_link.STL
Joints:
- joint joint1: limit lower=0.1 upper=4.15 effort=1000 velocity=10 -> lower=-2.09 upper=2.09 effort=1000 velocity=10
